File: hardware/OrangePi/OrangePiAdapter/OrangePiAdapter.sch (KiCad schematic (older format))
At the start: 14 parts

Commit message: Add buffer elco
Parts:
- added C1: 220u, symbol Device:CP
- gave numbers to parts that had none: 14
Connections:
- net labels removed: Enable, enable
- wire segments 42 -> 48
